Commit message: creating launch file for RTAB-Map

File: src/my_robot/urdf/my_robot.xacro (robot description, xacro)
@@ -66,4 +66,34 @@
     </collision>
   </link>
+<!-- adding RGB-D-->
+  <joint name="camera_optical_joint" type="fixed">
+    <origin xyz="0 0 0" rpy="-1.5707 0 -1.5707"/>
+    <parent link="camera"/>
+    <child link="camera_link_optical"/>
+    <axis xyz="0 1 0" rpy="0 0 0"/>
+  </joint>
+  <link name="camera_link_optical">
+    <inertial>
+      <origin xyz="0 0 0" rpy="0 0 0"/>
+      <mass value="0.1"/>
+        <inertia
+          ixx="1e-6" ixy="0" ixz="0"
+          iyy="1e-6" iyz="0"
+          izz="1e-6"
+      />
+    </inertial>
+    <visual>
+      <origin xyz="0 0 0" rpy="0 0 0"/>
+      <geometry>
+        <box size="0.05 0.05 0.05"/>
+      </geometry>
+    </visual>
+    <collision>
+      <origin xyz="0 0 0" rpy="0 0 0"/>
+      <geometry>
+        <box size="0.05 0.05 0.05"/>
+      </geometry>
+    </collision>
+  </link>
   <joint name="left_wheel_hinge" type="continuous">
     <origin xyz="0 0.15 0" rpy="0 0 0" />

Commit message: configuration map launch file

File: src/my_robot/urdf/my_robot.xacro (robot description, xacro)
@@ -73,27 +73,5 @@
     <axis xyz="0 1 0" rpy="0 0 0"/>
   </joint>
-  <link name="camera_link_optical">
-    <inertial>
-      <origin xyz="0 0 0" rpy="0 0 0"/>
-      <mass value="0.1"/>
-        <inertia
-          ixx="1e-6" ixy="0" ixz="0"
-          iyy="1e-6" iyz="0"
-          izz="1e-6"
-      />
-    </inertial>
-    <visual>
-      <origin xyz="0 0 0" rpy="0 0 0"/>
-      <geometry>
-        <box size="0.05 0.05 0.05"/>
-      </geometry>
-    </visual>
-    <collision>
-      <origin xyz="0 0 0" rpy="0 0 0"/>
-      <geometry>
-        <box size="0.05 0.05 0.05"/>
-      </geometry>
-    </collision>
-  </link>
+  <link name="camera_link_optical"></link>
   <joint name="left_wheel_hinge" type="continuous">
     <origin xyz="0 0.15 0" rpy="0 0 0" />
